Commit message: bugs added

File: erl2/urdf/m2wr_arm2.xacro (robot description, xacro)
@@ -1,6 +1,6 @@
 <?xml version="1.0" ?>
-<robot name="cluedo_robot" xmlns:xacro="https://www.ros.org/wiki/xacro" >
+<robot name="m2wr" xmlns:xacro="https://www.ros.org/wiki/xacro" >
  <xacro:include filename="$(find erl2)/urdf/materials.xacro" />
- <xacro:include filename="$(find erl2)/urdf/cluedo_robot.gazebo" />
+ <xacro:include filename="$(find erl2)/urdf/m2wr_arm2.gazebo" />
  <xacro:macro name="cylinder_inertia" params="mass r l">
     <inertia ixx="${mass*(3*r*r+l*l)/12}" ixy = "0" ixz = "0"
@@ -42,5 +42,5 @@
     <pose>0 0 0.1 0 0 0</pose>
     <inertial>
-      <mass value="7"/>
+      <mass value="5"/>
       <origin rpy="0 0 0" xyz="0 0 0.1"/>
       <inertia ixx="0.0395416666667" ixy="0" ixz="0" iyy="0.106208333333" iyz="0" izz="0.106208333333"/>
@@ -115,5 +115,5 @@
   <link name="arm_base_link">
   	<inertial>
-  		<mass value="0.5"/>
+  		<mass value="0.1"/>
   		<origin xyz="0 0 0" rpy="0 0 0" />
   		<inertia ixx="0.0000416666667" ixy="0" ixz="0" iyy="0.0000416666667" iyz="0" izz="0.0000416666667"/>
@@ -140,18 +140,19 @@
   <link name="arm_link_01">
   	<inertial>
-  		<mass value="0.015"/>
-  		<origin xyz="0 0 0" rpy="0 0 0" />
-  		<inertia ixx="0.000010279" ixy="0" ixz="0" iyy="0.000010279" iyz="0" izz="0.000007225"/>
-  	</inertial>
-  	<collision>
-  	  <origin xyz="0 0 0.25" rpy="0 0 0"/>
-      <geometry>
-        <cylinder radius="0.04" length="0.5"/>
-      </geometry>
-  	</collision>
-  	<visual>
-  	  <origin xyz="0 0 0.25" rpy="0 0 0"/>
-      <geometry>
-        <cylinder radius="0.04" length="0.5"/>
+  		<mass value="0.01"/>
+  		<origin xyz="0 0 0" rpy="0 0 0" />
+  		<xacro:cylinder_inertia mass="0.05" r="0.04" l="0.4" />
+  		<!--inertia ixx="0.000010279" ixy="0" ixz="0" iyy="0.000010279" iyz="0" izz="0.000007225"/-->
+  	</inertial>
+  	<collision>
+  	  <origin xyz="0 0 0.2" rpy="0 0 0"/>
+      <geometry>
+        <cylinder radius="0.04" length="0.4"/>
+      </geometry>
+  	</collision>
+  	<visual>
+  	  <origin xyz="0 0 0.2" rpy="0 0 0"/>
+      <geometry>
+        <cylinder radius="0.04" length="0.4"/>
       </geometry>
       <material name="red" />
@@ -160,5 +161,5 @@
   <joint name="arm_joint_01" type="revolute">
   	<axis xyz="0 0 1"/>
-  	<limit effort="1000.0" lower="-3.14" upper="3.14" velocity="0.2"/>
+  	<limit effort="10000.0" lower="-3.14" upper="3.14" velocity="0.2"/>
   	<origin rpy="0 0 0" xyz="0 0 0.05"/>
   	<parent link="arm_base_link"/>
@@ -167,18 +168,19 @@
     <link name="arm_link_02">
   	<inertial>
-  		<mass value="0.015"/>
-  		<origin xyz="0 0 0" rpy="0 0 0" />
-  		<inertia ixx="0.000010279" ixy="0" ixz="0" iyy="0.000010279" iyz="0" izz="0.000007225"/>
-  	</inertial>
-  	<collision>
-  	  <origin xyz="0 0 0.2" rpy="0 0 0"/>
-      <geometry>
-        <cylinder radius="0.04" length="0.5"/>
-      </geometry>
-  	</collision>
-  	<visual>
-  	  <origin xyz="0 0 0.25" rpy="0 0 0"/>
-      <geometry>
-        <cylinder radius="0.04" length="0.5"/>
+  		<mass value="0.01"/>
+  		<origin xyz="0 0 0" rpy="0 0 0" />
+  		<xacro:cylinder_inertia mass="0.05" r="0.04" l="0.4" />
+  		<!--inertia ixx="0.000010279" ixy="0" ixz="0" iyy="0.000010279" iyz="0" izz="0.000007225"/-->
+  	</inertial>
+  	<collision>
+  	  <origin xyz="0 0 0.2" rpy="0 0 0"/>
+      <geometry>
+        <cylinder radius="0.04" length="0.4"/>
+      </geometry>
+  	</collision>
+  	<visual>
+  	  <origin xyz="0 0 0.2" rpy="0 0 0"/>
+      <geometry>
+        <cylinder radius="0.04" length="0.4"/>
       </geometry>
       <material name="red" />
@@ -187,6 +189,6 @@
   <joint name="arm_joint_02" type="revolute">
   	<axis xyz="1 0 0"/>
-  	<limit effort="1000.0" lower="-1.8" upper="1.8" velocity="0.2"/>
-  	<origin rpy="0 0 0" xyz="0 0 0.5"/>
+  	<limit effort="10000.0" lower="-1.8" upper="1.8" velocity="0.2"/>
+  	<origin rpy="0 0 0" xyz="0 0 0.4"/>
   	<parent link="arm_link_01"/>
   	<child link="arm_link_02"/>
@@ -194,18 +196,19 @@
       <link name="arm_link_03">
   	<inertial>
-  		<mass value="0.015"/>
-  		<origin xyz="0 0 0" rpy="0 0 0" />
-  		<inertia ixx="0.000010279" ixy="0" ixz="0" iyy="0.000010279" iyz="0" izz="0.000007225"/>
-  	</inertial>
-  	<collision>
-  	  <origin xyz="0 0 0.2" rpy="0 0 0"/>
-      <geometry>
-        <cylinder radius="0.04" length="0.5"/>
-      </geometry>
-  	</collision>
-  	<visual>
-  	  <origin xyz="0 0 0.25" rpy="0 0 0"/>
-      <geometry>
-        <cylinder radius="0.04" length="0.5"/>
+  		<mass value="0.01"/>
+  		<origin xyz="0 0 0" rpy="0 0 0" />
+  		<xacro:cylinder_inertia mass="0.05" r="0.04" l="0.4" />
+  		<!--inertia ixx="0.000010279" ixy="0" ixz="0" iyy="0.000010279" iyz="0" izz="0.000007225"/-->
+  	</inertial>
+  	<collision>
+  	  <origin xyz="0 0 0.2" rpy="0 0 0"/>
+      <geometry>
+        <cylinder radius="0.04" length="0.4"/>
+      </geometry>
+  	</collision>
+  	<visual>
+  	  <origin xyz="0 0 0.2" rpy="0 0 0"/>
+      <geometry>
+        <cylinder radius="0.04" length="0.4"/>
       </geometry>
       <material name="red" />
@@ -214,6 +217,6 @@
   <joint name="arm_joint_03" type="revolute">
   	<axis xyz="1 0 0"/>
-  	<limit effort="1000.0" lower="-1.8" upper="1.8" velocity="0.2"/>
-  	<origin rpy="0 0 0" xyz="0 0 0.5"/>
+  	<limit effort="10000.0" lower="-1.8" upper="1.8" velocity="0.2"/>
+  	<origin rpy="0 0 0" xyz="0 0 0.4"/>
   	<parent link="arm_link_02"/>
   	<child link="arm_link_03"/>
@@ -221,10 +224,10 @@
     <link name="cluedo_link">
   	<inertial>
-  		<mass value="0.005"/>
+  		<mass value="0.01"/>
   		<origin xyz="0 0 0" rpy="0 0 0" />
   		<inertia ixx="0.000010279" ixy="0" ixz="0" iyy="0.000010279" iyz="0" izz="0.000007225"/>
   	</inertial>
   	<collision>
-  	  <origin xyz="0 0 0" rpy="0 0 1.57"/>
+  	  <origin xyz="0 0 0.04" rpy="0 0 1.57"/>
       <geometry>
         <box size="0.034 0.2 0.08"/>
@@ -241,6 +244,6 @@
   <joint name="arm_joint_04" type="revolute">
   	<axis xyz="1 0 0"/>
-  	<limit effort="1000.0" lower="-1.8" upper="1.8" velocity="0.5"/>
-  	<origin rpy="0 0 0" xyz="0 0 0.5"/>
+  	<limit effort="10000.0" lower="-1.8" upper="1.8" velocity="0.5"/>
+  	<origin rpy="0 0 0" xyz="0 0 0.4"/>
   	<parent link="arm_link_03"/>
   	<child link="cluedo_link"/>
@@ -248,5 +251,5 @@
 <link name="right_grip_link">
   	<inertial>
-  		<mass value="0.001"/>
+  		<mass value="0.01"/>
   		<origin xyz="0 0 0" rpy="0 0 0" />
   		<inertia ixx="0.000010279" ixy="0" ixz="0" iyy="0.000010279" iyz="0" izz="0.000007225"/>
@@ -275,5 +278,5 @@
   <link name="left_grip_link">
   	<inertial>
-  		<mass value="0.001"/>
+  		<mass value="0.01"/>
   		<origin xyz="0 0 0" rpy="0 0 0" />
   		<inertia ixx="0.000010279" ixy="0" ixz="0" iyy="0.000010279" iyz="0" izz="0.000007225"/>

File: erl2/urdf/materials.xacro (robot description, xacro)
@@ -1,4 +1,4 @@
 <?xml version="1.0" ?>
-<robot name="cluedo_robot" xmlns:xacro="https://www.ros.org/wiki/xacro" >
+<robot name="m2wr" xmlns:xacro="https://www.ros.org/wiki/xacro" >
   <material name="black">
     <color rgba="0.0 0.0 0.0 1.0"/>

File: erl2/urdf/robot2.urdf (robot description, URDF)
Before this commit: robot cluedo_robot, 11 links, 10 joints
Links:
- link arm_base_link: mass 0.5 -> 0.1
- link arm_link_01: mass 0.015 -> 0.01; geometry collision cylinder length=0.4 radius=0.04; visual cylinder length=0.4 radius=0.04
- link arm_link_02: mass 0.015 -> 0.01; geometry collision cylinder length=0.4 radius=0.04; visual cylinder length=0.4 radius=0.04
- link arm_link_03: mass 0.015 -> 0.01; geometry collision cylinder length=0.4 radius=0.04; visual cylinder length=0.4 radius=0.04
- link base_link: mass 7 -> 5
- link cluedo_link: mass 0.005 -> 0.01
- link left_grip_link: mass 0.001 -> 0.01
- link right_grip_link: mass 0.001 -> 0.01
Joints:
- joint arm_joint_01: limit lower=-3.14 upper=3.14 effort=1000.0 velocity=0.2 -> lower=-3.14 upper=3.14 effort=10000.0 velocity=0.2
- joint arm_joint_02: limit lower=-1.8 upper=1.8 effort=1000.0 velocity=0.2 -> lower=-1.8 upper=1.8 effort=10000.0 velocity=0.2; origin xyz=0 0 0.5 rpy=0 0 0 -> xyz=0 0 0.4 rpy=0 0 0
- joint arm_joint_03: limit lower=-1.8 upper=1.8 effort=1000.0 velocity=0.2 -> lower=-1.8 upper=1.8 effort=10000.0 velocity=0.2; origin xyz=0 0 0.5 rpy=0 0 0 -> xyz=0 0 0.4 rpy=0 0 0
- joint arm_joint_04: limit lower=-1.8 upper=1.8 effort=1000.0 velocity=0.5 -> lower=-1.8 upper=1.8 effort=10000.0 velocity=0.5; origin xyz=0 0 0.5 rpy=0 0 0 -> xyz=0 0 0.4 rpy=0 0 0
